File: hardware/src/bottom/53xLIDAR.kicad_pcb (KiCad board)
At the start: 2 copper layers, 75.4 x 75.4 mm, 53 parts, among them J1 CONN_01X06, J10 CONN_01X06, J11 CONN_01X06, J12 CONN_01X06, J13 CONN_01X06, J14 CONN_01X06, J15 CONN_01X06, J16 CONN_01X06, J17 USB_OTG, J18 UART_EXT, J19 I2C1_DEBUG, J2 CONN_01X06, J20 I2C2_DEBUG, J21 UART_DEBUG, J22 SWD, J23 SPI1_EXT, J3 CONN_01X06, J4 CONN_01X06, J5 CONN_01X06, J6 CONN_01X06, J7 CONN_01X06, J8 CONN_01X06, J9 CONN_01X06, U1 WS2812S, U2 WS2812S, U3 WS2812S, U4 WS2812S, U5 STM32F411RETx, U6 MPU-9250, U7 KF33_DPAK, Y1 24MHz SR PASSIVES 3225-24M-SR

Commit message: added LSM9DS1, revision 1
Parts:
- added C16: 4.7u, Capacitors_SMD:C_0805_HandSoldering, F.Cu at (173.5, 63.6)
- added C17: 100n, Capacitors_SMD:C_0402, F.Cu at (141.9, 71.1)
- added C18: 4.7u, Capacitors_SMD:C_0805_HandSoldering, F.Cu at (145.7, 69.8)
- added C19: 4.7u, Capacitors_SMD:C_0805_HandSoldering, F.Cu at (144.0, 69.8)
- added C20: 100n, Capacitors_SMD:C_0402, F.Cu at (141.0, 71.1)
- added C21: 10n 16V, Capacitors_SMD:C_0805_HandSoldering, F.Cu at (147.5, 69.8)
- added C22: 100n, Capacitors_SMD:C_0402, F.Cu at (142.7, 71.1)
- added J25: GS3, Connectors:GS3, F.Cu at (148.1, 74.6)
- added U8: LSM9DS1, Housings_LGA:LGA-24L_3x3.5mm_Pitch0.43mm, F.Cu at (144.1, 74.8)
- C14: value 1u -> 4.7u
- C15, C9: value 2.2u -> 4.7u
- R1: footprint Resistors_SMD:R_0603 -> Resistors_SMD:R_0402
- moved REF*** 8.44 mm to (132.2, 72.7)
- moved REF*** 3.91 mm to (143.0, 59.4)
- moved C15 2.07 mm to (173.5, 65.4)
Connections:
- U5 pad 34: (no net) -> IMU_DRDY_MAG
- U5 pad 51: (no net) -> IMU_INT_MAG
- U5 pad 52: (no net) -> IMU_CS_MAG
Routing:
- net IMU_DRDY_MAG: track 0.00 -> 60.6 mm, vias 0 -> 4
- net IMU_CS_MAG: track 0.00 -> 49.4 mm, vias 0 -> 4
- net IMU_INT_MAG: track 0.00 -> 46.4 mm, vias 0 -> 4
- net +3V3: track 40.0 -> 64.2 mm, vias 27 -> 33
- net IMU_CS: track 15.5 -> 38.9 mm, vias 0 -> 2
- net IMU_INT: track 27.4 -> 42.6 mm, vias 0 -> 2
- net Net-(C21-Pad2): track 0.00 -> 4.53 mm
- net SPI1_MISO: track 48.7 -> 53.1 mm, vias 1 -> 2
- net INT15: track 47.4 -> 43.7 mm
- net SDA_IMU: track 49.2 -> 52.7 mm, vias 3 -> 4
- net EXT_CS: track 53.1 -> 49.8 mm
- net SCL_IMU: track 56.1 -> 59.2 mm
- net Net-(J25-Pad2): track 0.00 -> 3.05 mm
- net SWDIO_PROGRAMMING: track 31.1 -> 33.7 mm
- net Net-(C22-Pad1): track 0.00 -> 2.12 mm
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Other:
- net class Default: via_dia 0.8 -> 0.4; via_drill 0.4 -> 0.2
- board text added: "DEN_A"
- board text added: "v1.r1 - Aug 18"
- board text removed: "v1.r0 - Jul 18"
