File: hardware/src/bottom/53xLIDAR.sch (KiCad schematic (older format))
At the start: 50 parts, among them J1 CONN_01X06, J10 CONN_01X06, J11 CONN_01X06, J12 CONN_01X06, J13 CONN_01X06, J14 CONN_01X06, J15 CONN_01X06, J16 CONN_01X06, J17 USB_OTG, J18 UART_EXT, J19 I2C1_DEBUG, J2 CONN_01X06, J20 I2C2_DEBUG, J21 UART_DEBUG, J22 SWD, J23 SPI1_EXT, J3 CONN_01X06, J4 CONN_01X06, J5 CONN_01X06, J6 CONN_01X06, J7 CONN_01X06, J8 CONN_01X06, J9 CONN_01X06, U1 WS2812S, U2 WS2812S, U3 WS2812S, U4 WS2812S, U5 STM32F411RETx, U6 MPU-9250, U7 KF33_DPAK, Y1 24MHz SR PASSIVES 3225-24M-SR

Commit message: added LSM9DS1, revision 1
Parts:
- removed WS1: WS2812S, symbol conn1:TEST_1P
- added C16, C18, C19: 4.7u, Capacitors_SMD:C_0805_HandSoldering, symbol device1:C
- added C17, C20: 100n, Capacitors_SMD:C_0402, symbol device1:C
- added C21: 10n 16V, Capacitors_SMD:C_0805_HandSoldering, symbol device1:C_Small
- added C22: 100n, Capacitors_SMD:C_0402, symbol device1:C_Small
- added J25: GS3, Connectors:GS3, symbol conn1:GS3
- added U8: LSM9DS1, Housings_LGA:LGA-24L_3x3.5mm_Pitch0.43mm, symbol Sensor_Motion:LSM9DS1
- C14: value 1u -> 4.7u
- C15, C9: value 2.2u -> 4.7u
Connections:
- net labels added: IMU_CS_MAG, IMU_DRDY_MAG, IMU_INT_MAG
- wire segments 345 -> 413
- no-connect marks 2 -> 3
