File: hardware/src/bottom/53xLIDAR.sch (KiCad schematic (older format))
At the start: 58 parts, among them J1 CONN_01X06, J10 CONN_01X06, J11 CONN_01X06, J12 CONN_01X06, J13 CONN_01X06, J14 CONN_01X06, J15 CONN_01X06, J16 CONN_01X06, J17 USB_OTG, J18 UART_EXT, J19 I2C1_DEBUG, J2 CONN_01X06, J20 I2C2_DEBUG, J21 UART_DEBUG, J22 SWD, J23 SPI1_EXT, J25 GS3, J3 CONN_01X06, J4 CONN_01X06, J5 CONN_01X06, J6 CONN_01X06, J7 CONN_01X06, J8 CONN_01X06, J9 CONN_01X06, U1 WS2812S, U2 WS2812S, U3 WS2812S, U4 WS2812S, U5 STM32F411RETx, U6 MPU-9250, U7 KF33_DPAK, U8 LSM9DS1, Y1 24MHz SR PASSIVES 3225-24M-SR

Commit message: Bom optimization
Parts:
- C1, C12, C13, C17, C2, C20, C22, C3, C4, C5, C6, C7, C8: footprint Capacitors_SMD:C_0402 -> Capacitors_SMD:C_0603
- C14, C15, C16, C18, C19, C21, C9: footprint Capacitors_SMD:C_0805_HandSoldering -> Capacitors_SMD:C_0603_HandSoldering
Changed lines of the file:
@@
 F 0 "C13" V 5046 7050 50  0000 C CNN
 F 1 "100n" V 5137 7050 50  0000 C CNN
-F 2 "Capacitors_SMD:C_0402" H 5275 7050 50  0001 C CNN
+F 2 "Capacitors_SMD:C_0603" H 5275 7050 50  0001 C CNN
 F 3 "~" H 5275 7050 50  0001 C CNN
 	1    5275 7050
@@
 F 0 "C12" H 5008 6004 50  0000 R CNN
 F 1 "100n" H 5008 6095 50  0000 R CNN
-F 2 "Capacitors_SMD:C_0402" H 5100 6050 50  0001 C CNN
+F 2 "Capacitors_SMD:C_0603" H 5100 6050 50  0001 C CNN
 F 3 "~" H 5100 6050 50  0001 C CNN
 	1    5100 6050
@@
 F 0 "C9" V 1925 2100 50  0000 C CNN
 F 1 "4.7u" V 1850 2175 50  0000 C CNN
-F 2 "Capacitors_SMD:C_0805_HandSoldering" H 1975 2200 50  0001 C CNN
+F 2 "Capacitors_SMD:C_0603_HandSoldering" H 1975 2200 50  0001 C CNN
 F 3 "~" H 1975 2200 50  0001 C CNN
 	1    1975 2200
@@
 F 0 "C15" H 5290 9346 50  0000 L CNN
 F 1 "4.7u" H 5290 9255 50  0000 L CNN
-F 2 "Capacitors_SMD:C_0805_HandSoldering" H 5213 9150 50  0001 C CNN
+F 2 "Capacitors_SMD:C_0603_HandSoldering" H 5213 9150 50  0001 C CNN
 F 3 "~" H 5175 9300 50  0001 C CNN
 	1    5175 9300
@@
 F 0 "C14" H 4040 9346 50  0000 L CNN
 F 1 "4.7u" H 4040 9255 50  0000 L CNN
-F 2 "Capacitors_SMD:C_0805_HandSoldering" H 3963 9150 50  0001 C CNN
+F 2 "Capacitors_SMD:C_0603_HandSoldering" H 3963 9150 50  0001 C CNN
 F 3 "~" H 3925 9300 50  0001 C CNN
 	1    3925 9300
@@
 F 0 "C5" H 1942 1046 50  0000 L CNN
 F 1 "100n" H 1942 955 50  0000 L CNN
-F 2 "Capacitors_SMD:C_0402" H 1850 1000 50  0001 C CNN
+F 2 "Capacitors_SMD:C_0603" H 1850 1000 50  0001 C CNN
 F 3 "~" H 1850 1000 50  0001 C CNN
 	1    1850 1000
@@
 F 0 "C6" H 2467 1046 50  0000 L CNN
 F 1 "100n" H 2467 955 50  0000 L CNN
-F 2 "Capacitors_SMD:C_0402" H 2375 1000 50  0001 C CNN
+F 2 "Capacitors_SMD:C_0603" H 2375 1000 50  0001 C CNN
 F 3 "~" H 2375 1000 50  0001 C CNN
 	1    2375 1000
@@
 F 0 "C7" H 2967 1046 50  0000 L CNN
 F 1 "100n" H 2967 955 50  0000 L CNN
-F 2 "Capacitors_SMD:C_0402" H 2875 1000 50  0001 C CNN
+F 2 "Capacitors_SMD:C_0603" H 2875 1000 50  0001 C CNN
 F 3 "~" H 2875 1000 50  0001 C CNN
 	1    2875 1000
@@
 F 0 "C8" H 3467 1046 50  0000 L CNN
 F 1 "100n" H 3467 955 50  0000 L CNN
-F 2 "Capacitors_SMD:C_0402" H 3375 1000 50  0001 C CNN
+F 2 "Capacitors_SMD:C_0603" H 3375 1000 50  0001 C CNN
 F 3 "~" H 3375 1000 50  0001 C CNN
 	1    3375 1000
@@
 F 0 "C1" H 9617 6271 50  0000 L CNN
 F 1 "100n" H 9617 6180 50  0000 L CNN
-F 2 "Capacitors_SMD:C_0402" H 9525 6225 50  0001 C CNN
+F 2 "Capacitors_SMD:C_0603" H 9525 6225 50  0001 C CNN
 F 3 "~" H 9525 6225 50  0001 C CNN
 	1    9525 6225
@@
 F 0 "C2" H 10142 6271 50  0000 L CNN
 F 1 "100n" H 10142 6180 50  0000 L CNN
-F 2 "Capacitors_SMD:C_0402" H 10050 6225 50  0001 C CNN
+F 2 "Capacitors_SMD:C_0603" H 10050 6225 50  0001 C CNN
 F 3 "~" H 10050 6225 50  0001 C CNN
 	1    10050 6225
@@
 F 0 "C3" H 10642 6271 50  0000 L CNN
 F 1 "100n" H 10642 6180 50  0000 L CNN
-F 2 "Capacitors_SMD:C_0402" H 10550 6225 50  0001 C CNN
+F 2 "Capacitors_SMD:C_0603" H 10550 6225 50  0001 C CNN
 F 3 "~" H 10550 6225 50  0001 C CNN
 	1    10550 6225
@@
 F 0 "C4" H 11142 6271 50  0000 L CNN
 F 1 "100n" H 11142 6180 50  0000 L CNN
-F 2 "Capacitors_SMD:C_0402" H 11050 6225 50  0001 C CNN
+F 2 "Capacitors_SMD:C_0603" H 11050 6225 50  0001 C CNN
 F 3 "~" H 11050 6225 50  0001 C CNN
 	1    11050 6225
@@
 F 0 "C17" H 9940 8346 50  0000 L CNN
 F 1 "100n" H 9940 8255 50  0000 L CNN
-F 2 "Capacitors_SMD:C_0402" H 9863 8150 50  0001 C CNN
+F 2 "Capacitors_SMD:C_0603" H 9863 8150 50  0001 C CNN
 F 3 "~" H 9825 8300 50  0001 C CNN
 	1    9825 8300
@@
 F 0 "C19" H 10715 8346 50  0000 L CNN
 F 1 "4.7u" H 10715 8255 50  0000 L CNN
-F 2 "Capacitors_SMD:C_0805_HandSoldering" H 10638 8150 50  0001 C CNN
+F 2 "Capacitors_SMD:C_0603_HandSoldering" H 10638 8150 50  0001 C CNN
 F 3 "~" H 10600 8300 50  0001 C CNN
 	1    10600 8300
@@
 F 0 "C18" H 10340 8346 50  0000 L CNN
 F 1 "4.7u" H 10340 8255 50  0000 L CNN
-F 2 "Capacitors_SMD:C_0805_HandSoldering" H 10263 8150 50  0001 C CNN
+F 2 "Capacitors_SMD:C_0603_HandSoldering" H 10263 8150 50  0001 C CNN
 F 3 "~" H 10225 8300 50  0001 C CNN
 	1    10225 8300
@@
 F 0 "C20" H 8235 8279 50  0000 R CNN
 F 1 "100n" H 8235 8370 50  0000 R CNN
-F 2 "Capacitors_SMD:C_0402" H 8388 8175 50  0001 C CNN
+F 2 "Capacitors_SMD:C_0603" H 8388 8175 50  0001 C CNN
 F 3 "~" H 8350 8325 50  0001 C CNN
 	1    8350 8325
@@
 F 0 "C16" H 5690 9346 50  0000 L CNN
 F 1 "4.7u" H 5690 9255 50  0000 L CNN
-F 2 "Capacitors_SMD:C_0805_HandSoldering" H 5613 9150 50  0001 C CNN
+F 2 "Capacitors_SMD:C_0603_HandSoldering" H 5613 9150 50  0001 C CNN
 F 3 "~" H 5575 9300 50  0001 C CNN
 	1    5575 9300
@@
 F 0 "C21" H 8250 9850 50  0000 R CNN
 F 1 "10n 16V" H 8300 9975 50  0000 R CNN
-F 2 "Capacitors_SMD:C_0805_HandSoldering" H 7900 9900 50  0001 C CNN
+F 2 "Capacitors_SMD:C_0603_HandSoldering" H 7900 9900 50  0001 C CNN
 F 3 "~" H 7900 9900 50  0001 C CNN
 	1    7900 9900
@@
 F 0 "C22" H 8292 9946 50  0000 L CNN
 F 1 "100n" H 8292 9855 50  0000 L CNN
-F 2 "Capacitors_SMD:C_0402" H 8200 9900 50  0001 C CNN
+F 2 "Capacitors_SMD:C_0603" H 8200 9900 50  0001 C CNN
 F 3 "~" H 8200 9900 50  0001 C CNN
 	1    8200 9900
