File: hardware/src/top/TopPcb.kicad_pcb (KiCad board)
At the start: 2 copper layers, 75.4 x 75.4 mm, 18 parts, among them J1 CONN_01X06, J10 CONN_01X06, J11 CONN_01X06, J12 CONN_01X06, J13 CONN_01X06, J14 CONN_01X06, J15 CONN_01X06, J16 CONN_01X06, J2 CONN_01X06, J3 CONN_01X06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

Commit message: fixed manufactury requirements
Other:
- board text added: "BOTTOM SOLDERMASK"
Changed lines of the file:
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@@
   (general
     (thickness 1.6)
-    (drawings 90)
+    (drawings 91)
     (tracks 291)
     (zones 0)
@@
       (drillshape 0)
       (scaleselection 1)
-      (outputdirectory ""))
+      (outputdirectory "../../gerbers/top/"))
   )
   (net 0 "")
@@
     )
     (fp_circle (center -3.25 -0.85) (end -3.179289 -0.85) (layer F.SilkS) (width 0.2))
-    (pad 5 smd rect (at 1.5 0.05 22.5) (size 0.5 1.2) (layers F.Cu F.Mask))
+    (pad 5 smd rect (at 1.499999 0.05 22.5) (size 0.5 1.2) (layers F.Cu F.Mask))
     (pad 4 smd rect (at 0.5 0.05 22.5) (size 0.5 1.2) (layers F.Cu F.Mask))
     (pad 3 smd rect (at -0.5 0.05 22.5) (size 0.5 1.2) (layers F.Cu F.Mask)
@@
     (pad 3 smd rect (at -0.5 0.05 67.5) (size 0.5 1.2) (layers F.Cu F.Mask)
       (net 4 SCL1))
-    (pad 2 smd rect (at -1.5 0.05 67.5) (size 0.5 1.2) (layers F.Cu F.Mask)
+    (pad 2 smd rect (at -1.499999 0.05 67.5) (size 0.5 1.2) (layers F.Cu F.Mask)
       (net 3 SDA1))
     (pad 6 smd rect (at 3.25 0.05 67.5) (size 1 1.2) (layers F.Cu F.Mask)
@@
     )
     (fp_circle (center -3.25 -0.85) (end -3.179289 -0.85) (layer F.SilkS) (width 0.2))
-    (pad 5 smd rect (at 1.5 0.05 112.5) (size 0.5 1.2) (layers F.Cu F.Mask))
+    (pad 5 smd rect (at 1.499999 0.05 112.5) (size 0.5 1.2) (layers F.Cu F.Mask))
     (pad 4 smd rect (at 0.5 0.05 112.5) (size 0.5 1.2) (layers F.Cu F.Mask))
     (pad 3 smd rect (at -0.5 0.05 112.5) (size 0.5 1.2) (layers F.Cu F.Mask)
@@
     (pad 3 smd rect (at -0.5 0.05 157.5) (size 0.5 1.2) (layers F.Cu F.Mask)
       (net 4 SCL1))
-    (pad 2 smd rect (at -1.5 0.05 157.5) (size 0.5 1.2) (layers F.Cu F.Mask)
+    (pad 2 smd rect (at -1.499999 0.05 157.5) (size 0.5 1.2) (layers F.Cu F.Mask)
       (net 3 SDA1))
     (pad 6 smd rect (at 3.25 0.05 157.5) (size 1 1.2) (layers F.Cu F.Mask)
@@
     )
     (fp_circle (center -3.25 -0.85) (end -3.179289 -0.85) (layer F.SilkS) (width 0.2))
-    (pad 5 smd rect (at 1.5 0.05 202.5) (size 0.5 1.2) (layers F.Cu F.Mask))
+    (pad 5 smd rect (at 1.499999 0.05 202.5) (size 0.5 1.2) (layers F.Cu F.Mask))
     (pad 4 smd rect (at 0.5 0.05 202.5) (size 0.5 1.2) (layers F.Cu F.Mask))
     (pad 3 smd rect (at -0.5 0.05 202.5) (size 0.5 1.2) (layers F.Cu F.Mask)
@@
     (pad 3 smd rect (at -0.5 0.05 247.5) (size 0.5 1.2) (layers F.Cu F.Mask)
       (net 5 SCL2))
-    (pad 2 smd rect (at -1.5 0.05 247.5) (size 0.5 1.2) (layers F.Cu F.Mask)
+    (pad 2 smd rect (at -1.499999 0.05 247.5) (size 0.5 1.2) (layers F.Cu F.Mask)
       (net 6 SDA2))
     (pad 6 smd rect (at 3.25 0.05 247.5) (size 1 1.2) (layers F.Cu F.Mask)
@@
     )
     (fp_circle (center -3.25 -0.85) (end -3.179289 -0.85) (layer F.SilkS) (width 0.2))
-    (pad 5 smd rect (at 1.5 0.05 292.5) (size 0.5 1.2) (layers F.Cu F.Mask))
+    (pad 5 smd rect (at 1.499999 0.05 292.5) (size 0.5 1.2) (layers F.Cu F.Mask))
     (pad 4 smd rect (at 0.5 0.05 292.5) (size 0.5 1.2) (layers F.Cu F.Mask))
     (pad 3 smd rect (at -0.5 0.05 292.5) (size 0.5 1.2) (layers F.Cu F.Mask)
@@
     (pad 3 smd rect (at -0.5 0.05 337.5) (size 0.5 1.2) (layers F.Cu F.Mask)
       (net 5 SCL2))
-    (pad 2 smd rect (at -1.5 0.05 337.5) (size 0.5 1.2) (layers F.Cu F.Mask)
+    (pad 2 smd rect (at -1.499999 0.05 337.5) (size 0.5 1.2) (layers F.Cu F.Mask)
       (net 6 SDA2))
     (pad 6 smd rect (at 3.25 0.05 337.5) (size 1 1.2) (layers F.Cu F.Mask)
@@
       (xy -3.43224 2.584467) (xy -3.324904 2.572722) (xy -3.231114 2.584505)) (layer F.SilkS) (width 0.01))
   )
+  (gr_text "BOTTOM SOLDERMASK" (at 158.88 34.89) (layer B.Mask)
+    (effects (font (size 1.5 1.5) (thickness 0.3)) (justify mirror))
+  )
   (gr_text 5N44P.github.io/53xLIDAR (at 158.2 54.7) (layer F.SilkS)

Commit message: Update TopPcb.kicad_pcb
Other:
- board text added: "valerionew.github.io/53xLIDAR"
- board text removed: "5N44P.github.io/53xLIDAR"
Changed lines of the file:
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@@
     (effects (font (size 1.5 1.5) (thickness 0.3)) (justify mirror))
   )
-  (gr_text 5N44P.github.io/53xLIDAR (at 158.2 54.7) (layer F.SilkS)
+  (gr_text valerionew.github.io/53xLIDAR (at 158.2 54.7) (layer F.SilkS)
     (effects (font (size 1 1) (thickness 0.15)))
   )
